Commit message: x1pro_rm001：手指碰撞按弧面分段，手指参数 100/20/摩擦 2.0
- 手指内侧是内凹弧面，单个凸包跨过它、最多悬空 5 mm；prepare 新增 SLABS，
  沿手指轴线等分 8 段各取凸包，间隙降到 0.5 mm 以内
- 手指驱动 100 N·m/rad、阻尼 20，指垫摩擦 (2.0, 1.6)；x1pro 的 author()
  可传入材料
- CPU、GPU 验收均 12/12；实时率与 x1pro、分段前在测量波动内

Co-Authored-By: Claude Opus 5.5 <noreply@anthropic.com>

File: asset_sources/robots/x1pro_rm001/robot.urdf (robot description, URDF)
Before this commit: robot ex001_robot, 79 links, 78 joints
Links:
- link left_arm_gripper_left_link: geometry collision mesh filename=meshes/collision/gripper_left_link_0.ply; collision mesh filename=meshes/collision/gripper_left_link_1.ply
- link left_arm_gripper_right_link: geometry collision mesh filename=meshes/collision/gripper_right_link_0.ply; collision mesh filename=meshes/collision/gripper_right_link_1.ply
- link right_arm_gripper_left_link: geometry collision mesh filename=meshes/collision/gripper_left_link_0.ply; collision mesh filename=meshes/collision/gripper_left_link_1.ply
- link right_arm_gripper_right_link: geometry collision mesh filename=meshes/collision/gripper_right_link_0.ply; collision mesh filename=meshes/collision/gripper_right_link_1.ply
