Commit message: x1pro：平面指垫、手指刚度 5000 与夹持推力验收用例
Co-Authored-By: Claude Opus 5.5 <noreply@anthropic.com>

File: asset_sources/robots/x1pro/robot.urdf (robot description, URDF)
Before this commit: robot ex001_robot, 79 links, 78 joints
Links:
- link left_arm_gripper_left_link: geometry collision box size=0.025 0.003 0.018; collision mesh filename=meshes/collision/gripper_left_link_0.ply
- link left_arm_gripper_right_link: geometry collision box size=0.025 0.003 0.018; collision mesh filename=meshes/collision/gripper_right_link_0.ply
- link right_arm_gripper_left_link: geometry collision box size=0.025 0.003 0.018; collision mesh filename=meshes/collision/gripper_left_link_0.ply
- link right_arm_gripper_right_link: geometry collision box size=0.025 0.003 0.018; collision mesh filename=meshes/collision/gripper_right_link_0.ply
